File: Luminometer_RPi/_autosave-Luminometer_RPi.kicad_pcb (KiCad board)
At the start: 4 copper layers, 75.2 x 50 mm, 57 parts, among them J1 PMIC_header_right_angle, J2 H2191-ND, J3 H2191-ND, J4 RPi_SocketHeader, J5 H2191-ND, J6 H2191-ND, J7 Harting_15110122601000, J8 H2191-ND, Q1 IRLML6344TRPBF, Q2 IRLML6344TRPBF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

Commit message: Make production files
- Fix ferrite bead part number
Other:
- rule pad_to_mask_clearance: 0 -> 0.0508
Changed lines of the file:
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@@
     (pad_size 0.8 1.1)
     (pad_drill 0)
-    (pad_to_mask_clearance 0)
+    (pad_to_mask_clearance 0.0508)
     (aux_axis_origin 106.5 61.5)
     (visible_elements 7FFFFE3F)
@@
       (padsonsilk true)
       (subtractmaskfromsilk false)
-      (outputformat 4)
+      (outputformat 1)
       (mirror false)
       (drillshape 0)
